Commit message: sarkofag visualization fix

File: sark_description/robots/sarkofag.urdf.xacro (robot description, xacro)
@@ -48,5 +48,14 @@
       <color rgba=".2 .2 .2 1" />
     </material>
-  </visual>
+    </visual>
+    <visual>
+      <origin rpy="0 1.57 0" xyz="0.09 0.0 0.90"/>
+      <geometry>
+         <cylinder radius="0.06" length="0.12"/>
+      </geometry>
+      <material name="gray">
+      <color rgba=".2 .2 .2 1" />
+    </material>
+    </visual>
   </link>
   <joint name="SarkofagJoint" type="revolute">
@@ -64,14 +73,19 @@
     </inertial>
     <visual>
-      <origin rpy="-1.57 0 0.0" xyz="0.2 0.0 0.2"/>
+      <origin rpy="-1.57 0 0.0" xyz="0.18 0.0 0.2"/>
       <geometry>
         <box size="0.02 0.8 0.04" />
       </geometry>
     </visual>
+    <visual>
+      <origin rpy="0 1.57 0" xyz="0.18 0.0 0.0"/>
+      <geometry>
+         <cylinder radius="0.06" length="0.06"/>
+      </geometry>
+    </visual>
     <collision>
-      <origin rpy="-1.57 0 0.0" xyz="0 0 0.4"/>
+      <origin rpy="-1.57 0 0.0" xyz="0.18 0 0.2"/>
       <geometry>
-        <!--<mesh filename="package://sark_description/meshes/link1.stlb" />-->
-	<box size="0.1 0.10 0.1"/>
+        <box size="0.02 0.8 0.04" />
       </geometry>
     </collision>

Commit message: urdf fix

File: sark_description/robots/sarkofag.urdf.xacro (robot description, xacro)
@@ -60,5 +60,5 @@
   </link>
   <joint name="SarkofagJoint" type="revolute">
-    <origin rpy="0 0 0" xyz="0.0 0.0 0.90"/>
+    <origin rpy="-2.6179 0 0" xyz="0.0 0.0 0.90"/>
     <axis xyz="1 0 0"/>
     <limit lower="-2.96705973" upper="2.96705973" effort="10.0" velocity="10.0" />

Commit message: kinematic upgrade, homing

File: sark_description/robots/sarkofag.urdf.xacro (robot description, xacro)
@@ -60,5 +60,5 @@
   </link>
   <joint name="SarkofagJoint" type="revolute">
-    <origin rpy="-2.6179 0 0" xyz="0.0 0.0 0.90"/>
+    <origin rpy="-1.57 0 0" xyz="0.0 0.0 0.90"/>
     <axis xyz="1 0 0"/>
     <limit lower="-2.96705973" upper="2.96705973" effort="10.0" velocity="10.0" />

Commit message: urdf fix

File: sark_description/robots/sarkofag.urdf.xacro (robot description, xacro)
@@ -5,5 +5,5 @@
        xmlns:xacro="http://ros.org/wiki/fixme"
        xmlns:interface="http://playerstage.sourceforge.net/gazebo/xmlschema/#interface">
-  <property name="M_PI" value="3.14159"/>
+  <xacro:property name="M_PI" value="3.14159"/>
   <link name="world">
     <!--<inertial>
